File: PCB/RF_R1_8-9Xu.kicad_pcb (KiCad board)
At the start: 4 copper layers, 353 x 151 mm, 181 parts, among them J1 JST, J2 JST, SW1 BOOT0, SW10 EC_SW, SW100 EC_SW, SW11 EC_SW, SW12 EC_SW, SW13 EC_SW, SW14 EC_SW, SW15 EC_SW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

Commit message: Update
Parts:
- turned SW69 to 90 degrees
Connections:
- SW55 pad 1: ROW3 -> COL0
- SW55 pad 2: COL0 -> ROW3
- SW70 pad 1: ROW4 -> COL0
- SW70 pad 2: COL0 -> ROW4
